Commit message: fixed bugs on ar tag boundles

File: urdf/ikea_chair_cushion.xacro (robot description, xacro)
@@ -38,10 +38,10 @@
 		<parent link="${link_name}" />
 		<child link = "${link_name}_hole_2_1" />
-		<origin xyz="-0.048 0.15 -0.007" rpy="0 ${pi} 0" />
+		<origin xyz="-0.048 0.146 -0.007" rpy="0 ${pi} 0" />
 	</joint>
 	<joint name="${link_name}_hole_2_2_joint" type="fixed">
 		<parent link="${link_name}" />
 		<child link = "${link_name}_hole_2_2" />
-		<origin xyz="0.048 0.15 -0.007" rpy="0 ${pi} 0" />
+		<origin xyz="0.048 0.146 -0.007" rpy="0 ${pi} 0" />
 	</joint>
 </xacro:macro>

File: urdf/ikea_chair_front_part.xacro (robot description, xacro)
@@ -50,10 +50,10 @@
 		<parent link="${link_name}" />
 		<child link = "${link_name}_hole_3_1" />
-		<origin xyz="-0.048 -0.0225 0.0" rpy="${pi/2} 0  0" />
+		<origin xyz="-0.048 0.0225 0.0" rpy="${-pi/2} 0  0" />
 	</joint>
 	<joint name="${link_name}_hole_3_2_joint" type="fixed">
 		<parent link="${link_name}" />
 		<child link = "${link_name}_hole_3_2" />
-		<origin xyz="0.048 -0.0225 0.0" rpy="${pi/2} 0 0" />
+		<origin xyz="0.048 0.0225 0.0" rpy="${-pi/2} 0 0" />
 	</joint>
 </xacro:macro>
